File: udb-s.kicad_sch (KiCad schematic)
At the start: 10 parts, among them J1 TYPE-C-31-M-12, J2 78171-0004, U1 TPD4E05U06DQAR

Commit message: Swap J2 Pico-EZmate for JST-SH compatible XYECONN XY-SH1.0-4A61
Same 1:1 pinout (5V, D-, D+, GND). Side-entry header sits where the
EZmate was, opening toward the board's inner edge. 5V/D-/D+ stubs
moved onto the 1.00 mm pins, F1's 5V via nudged 0.25 mm for clearance
to the new mounting pad, GND pour refilled. Files stay in KiCad 6
format.
Parts:
- J2: value 78171-0004 -> XY-SH1.0-4A61; footprint locallib:PicoEZMate-Reinforced-Lite -> locallib:XY-SH1.0-4A61; LCSC Part Number C588524 -> C19271998; Manufacturer MOLEX -> XYECONN; Manufacturer Part Number 78171-0004 -> XY-SH1.0-4A61
Other:
- note added: "JST-SH (XYECONN XY-SH1.0-4A61)"
- note removed: "Pico-EZMate"
Changed lines of the file:
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@@
     (effects (font (size 5.08 5.08)) (justify left bottom))
   )
-  (text "Pico-EZMate" (at 158.75 33.02 0)
+  (text "JST-SH (XYECONN XY-SH1.0-4A61)" (at 158.75 33.02 0)
     (effects (font (size 2.54 2.54)) (justify left bottom))
   )
@@
       (effects (font (size 1.27 1.27)) (justify left))
     )
-    (property "Value" "78171-0004" (id 1) (at 177.165 49.2505 0)
-      (effects (font (size 1.27 1.27)) (justify left))
-    )
-    (property "Footprint" "locallib:PicoEZMate-Reinforced-Lite" (id 2) (at 173.99 46.355 0)
+    (property "Value" "XY-SH1.0-4A61" (id 1) (at 177.165 49.2505 0)
+      (effects (font (size 1.27 1.27)) (justify left))
+    )
+    (property "Footprint" "locallib:XY-SH1.0-4A61" (id 2) (at 173.99 46.355 0)
       (effects (font (size 1.27 1.27)) hide)
     )
@@
       (effects (font (size 1.27 1.27)) hide)
     )
-    (property "Manufacturer" "MOLEX" (id 4) (at 173.99 46.355 0)
-      (effects (font (size 1.27 1.27)) hide)
-    )
-    (property "Manufacturer Part Number" "78171-0004" (id 5) (at 173.99 46.355 0)
-      (effects (font (size 1.27 1.27)) hide)
-    )
-    (property "LCSC Part Number" "C588524" (id 6) (at 173.99 46.355 0)
+    (property "Manufacturer" "XYECONN" (id 4) (at 173.99 46.355 0)
+      (effects (font (size 1.27 1.27)) hide)
+    )
+    (property "Manufacturer Part Number" "XY-SH1.0-4A61" (id 5) (at 173.99 46.355 0)
+      (effects (font (size 1.27 1.27)) hide)
+    )
+    (property "LCSC Part Number" "C19271998" (id 6) (at 173.99 46.355 0)
       (effects (font (size 1.27 1.27)) hide)
     )
@@
     )
     (path "/9bedc7ad-26a6-4dea-8309-3bb1cd87c5e7"
-      (reference "J2") (unit 1) (value "78171-0004") (footprint "locallib:PicoEZMate-Reinforced-Lite")
+      (reference "J2") (unit 1) (value "XY-SH1.0-4A61") (footprint "locallib:XY-SH1.0-4A61")
     )
     (path "/d199325f-3460-4780-9af2-504e32113c8b"
