File: udb-s.kicad_pcb (KiCad board)
At the start: 4 copper layers, 40 x 9 mm, 11 parts, among them J1 TYPE-C-31-M-12, J2 XY-SH1.0-4A61, U1 TPD4E05U06DQAR

Commit message: Reinforce J2 mounting pads; S1-SH silkscreen
J2's mounting pads get a B.Cu mirror and three 0.6/0.3 plated holes
each, as on the EZmate footprint (0.3 drill keeps 0.15 annular ring).
Silkscreen: front reads 'JST-SH 1:1' and the J2 pin order, board name
'Unified-S1-SH'; back carries 'Unified-S1-SH V1.1' and this repo URL.
GND pour refilled.
Other:
- board text added: "5V D- D+ G"
- board text added: "JST-SH 1:1"
- board text added: "Unified-S1-SH"
- board text added: "Unified-S1-SH V1.1 github.com/ dubnubdubnub/ UDB-S-SH"
- board text removed: "USE ONLY uDB CABLES"
- board text removed: "Unified-S1 V1.1"
- board text removed: "Unified-S1 V1.1 www.unified- daughterboard.github.io"
Changed lines of the file:
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@@
     (pad "MP" smd rect (at 2.8 2) (size 1.2 2) (layers "F.Cu" "F.Paste" "F.Mask")
       (net 1 "GND") (pinfunction "MountPin") (pintype "passive"))
+    (pad "MP" smd rect (at -2.8 2) (size 1.2 2) (layers "B.Cu") (net 1 "GND") (pinfunction "MountPin") (pintype "passive"))
+    (pad "MP" thru_hole circle (at -2.8 1.4) (size 0.6 0.6) (drill 0.3) (layers *.Cu) (net 1 "GND") (pinfunction "MountPin") (pintype "passive"))
+    (pad "MP" thru_hole circle (at -2.8 2.0) (size 0.6 0.6) (drill 0.3) (layers *.Cu) (net 1 "GND") (pinfunction "MountPin") (pintype "passive"))
+    (pad "MP" thru_hole circle (at -2.8 2.6) (size 0.6 0.6) (drill 0.3) (layers *.Cu) (net 1 "GND") (pinfunction "MountPin") (pintype "passive"))
+    (pad "MP" smd rect (at 2.8 2) (size 1.2 2) (layers "B.Cu") (net 1 "GND") (pinfunction "MountPin") (pintype "passive"))
+    (pad "MP" thru_hole circle (at 2.8 1.4) (size 0.6 0.6) (drill 0.3) (layers *.Cu) (net 1 "GND") (pinfunction "MountPin") (pintype "passive"))
+    (pad "MP" thru_hole circle (at 2.8 2.0) (size 0.6 0.6) (drill 0.3) (layers *.Cu) (net 1 "GND") (pinfunction "MountPin") (pintype "passive"))
+    (pad "MP" thru_hole circle (at 2.8 2.6) (size 0.6 0.6) (drill 0.3) (layers *.Cu) (net 1 "GND") (pinfunction "MountPin") (pintype "passive"))
     (model "${KIPRJMOD}/libraries/locallib.pretty/XY-SH1.0-4A61.step"
       (offset (xyz 0 -0.65 3.1))
@@
   (gr_line (start 147 90.5) (end 116 90.499999) (layer "Edge.Cuts") (width 0.1))
   (gr_line (start 116 99.500001) (end 147 99.5) (layer "Edge.Cuts") (width 0.1))
-  (gr_text "Unified-S1 V1.1\nwww.unified-\ndaughterboard.github.io" (at 126.25 95) (layer "B.SilkS")
+  (gr_text "Unified-S1-SH V1.1\ngithub.com/\ndubnubdubnub/\nUDB-S-SH" (at 126.25 94.6) (layer "B.SilkS")
     (effects (font (size 0.8 0.8) (thickness 0.2)) (justify mirror))
   )
-  (gr_text "USE ONLY\nuDB CABLES" (at 122 91.95) (layer "F.SilkS")
+  (gr_text "JST-SH 1:1" (at 122 91.25) (layer "F.SilkS")
+    (effects (font (size 0.8 0.8) (thickness 0.15)))
+  )
+  (gr_text "5V D- D+ G" (at 122 92.55) (layer "F.SilkS")
+    (effects (font (size 0.8 0.8) (thickness 0.15)))
+  )
+  (gr_text "Unified-S1-SH" (at 139.1 98.5) (layer "F.SilkS")
     (effects (font (size 0.8 0.8) (thickness 0.2)))
   )
-  (gr_text "Unified-S1 V1.1" (at 139.1 98.5) (layer "F.SilkS")
-    (effects (font (size 0.8 0.8) (thickness 0.2)))
-  )
